File: handcart V6.kicad_pcb (KiCad board)
At the start: 2 copper layers, 115 parts, among them J1 Conn_01x05, J10 Conn_02x03_Odd_Even, J11 Conn_01x03, J12 Conn_01x04, J13 Conn_01x04, J132 TE_Ampseal_23, J14 Conn_01x03, J15 Conn_01x02, J16 Conn_01x02, J17 Conn_01x02, J18 Conn_01x02, J19 Raspberry_Pi_2_3, J2 Conn_01x02, J20 Conn_01x02, J21 Conn_01x02, J22 DB9_Female_DCE, J23 Conn_02x05, J24 TE_AmpSeal_14_776273-1, J25 Conn_02x06_Top_Bottom, J3 Conn_01x02, J4 Conn_01x02, J5 Conn_01x02, J6 Conn_01x02, J7 Conn_01x02, J8 Conn_01x02, J9 Conn_01x02, K1 EX12U1S, Q1 2N7002NXAK, Q10 2N7002NXAK, Q11 2N7002NXAK, Q12 2N7002NXAKR, Q13 NTR5105PT1G, Q14 2N7002NXAKR, Q15 2N7002NXAK, Q2 NTR5105PT1G, Q3 NTR5105PT1G, Q4 2N7002NXAK, Q5 2N7002NXAK, Q6 2N7002NXAK, Q7 2N7002NXAK, Q8 2N7002NXAK, Q9 2N7002NXAK, SW1 SW_SPDT, U1 Tex_DCDC_v2, U2 DCDC2510, U3 PCA9634PW,118, U4 MCP2515-xSO, U5 MCP2562-E-SN, U6 MAX3232CDR, Y1 16MHz

Commit message: Changed mosfet, fixed all the datasheets, added 3D models
Parts:
- added Q6: 2N7002NXAK, Package_TO_SOT_SMD:SOT-23, F.Cu at (257.8, 75.2)
- J10: footprint Connector_Molex:Molex_Micro-Fit_3.0_43045-0600_2x03_P3.00mm_Horizontal -> Connector_Molex:Molex_Micro-Fit_3.0_43045-0612_2x03_P3.00mm_Vertical
- J14: footprint Connector_Molex:Molex_Micro-Fit_3.0_43650-0300_1x03_P3.00mm_Horizontal -> Connector_Molex:Molex_Micro-Fit_3.0_43650-0315_1x03_P3.00mm_Vertical
- J23, J25: footprint Connector_Molex:Molex_Micro-Fit_3.0_43045-1000_2x05_P3.00mm_Horizontal -> Connector_Molex:Molex_Micro-Fit_3.0_43045-1012_2x05_P3.00mm_Vertical
- Q10, Q11, Q4, Q5, Q7, Q8, Q9: value 2N7002NXAK -> SSM3K361TU,LF; footprint Package_TO_SOT_SMD:SOT-23 -> 00_proj-lib:SOTFL65P210X75-3N
- Q14: value 2N7002NXAKR -> SSM3K361TU,LF; footprint Package_TO_SOT_SMD:SOT-23 -> 00_proj-lib:SOTFL65P210X75-3N
- moved J11 403.4 mm to (276.6, 200.5), turned to 180 degrees
- moved J6 392.8 mm to (333.7, 170.0)
- moved J2 391.0 mm to (319.8, 170.0)
- moved J12 387.3 mm to (260.8, 200.3), turned to 180 degrees
- moved J8 383.8 mm to (266.4, 176.3), turned to 90 degrees
- moved J13 383.1 mm to (241.7, 200.3), turned to 180 degrees
- moved JP1 377.5 mm to (296.8, 154.4)
- moved J15 360.2 mm to (252.5, 176.3), turned to 90 degrees
- moved J21 358.3 mm to (187.7, 168.7), turned to 90 degrees
- moved J17 335.7 mm to (222.0, 176.3), turned to 90 degrees
- moved J7 334.7 mm to (238.5, 176.3), turned to 90 degrees
- moved J10 332.3 mm to (172.0, 164.3)
- moved J18 327.0 mm to (303.0, 115.5)
- moved J16 326.7 mm to (208.0, 176.3), turned to 90 degrees
- moved J1 322.8 mm to (209.6, 116.2)
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Connections:
- R33 pad 1: Net-(Q6-Pad1) -> Net-(R33-Pad1)
- R34 pad 1: Net-(Q6-Pad1) -> Net-(R33-Pad1)
