File: RS_232.kicad_sch (KiCad schematic)
At the start: 10 parts, among them J22 DB9_Female_DCE, SW1 SW_SPDT, U6 MAX3232CDR

Commit message: Major changes after the schematic review. Refer to Github for all the changes
Parts:
- J26: renamed from J22; value DB9_Female_DCE -> RS_232
- renumbered R37 to R36, R38 to R37
Changed lines of the file:
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@@
   (symbol (lib_id "power:+3.3V") (at 121.285 74.93 0) (mirror y) (unit 1)
     (in_bom yes) (on_board yes)
-    (property "Reference" "#PWR0174" (id 0) (at 121.285 78.74 0)
+    (property "Reference" "#PWR076" (id 0) (at 121.285 78.74 0)
       (effects (font (size 1.27 1.27)) hide)
     )
@@
   (symbol (lib_id "power:GND") (at 168.91 129.54 90) (unit 1)
     (in_bom yes) (on_board yes)
-    (property "Reference" "#PWR0179" (id 0) (at 175.26 129.54 0)
+    (property "Reference" "#PWR080" (id 0) (at 175.26 129.54 0)
       (effects (font (size 1.27 1.27)) hide)
     )
@@
   (symbol (lib_id "Device:R") (at 123.825 80.01 0) (unit 1)
     (in_bom yes) (on_board yes)
-    (property "Reference" "R38" (id 0) (at 121.285 81.28 90)
-      (effects (font (size 1.27 1.27)) (justify left))
-    )
-    (property "Value" "10k" (id 1) (at 123.825 81.915 90)
+    (property "Reference" "R37" (id 0) (at 125.73 78.74 0)
+      (effects (font (size 1.27 1.27)) (justify left))
+    )
+    (property "Value" "10k" (id 1) (at 125.73 81.28 0)
       (effects (font (size 1.27 1.27)) (justify left))
     )
@@
   (symbol (lib_id "power:+3.3V") (at 147.955 41.275 0) (mirror y) (unit 1)
     (in_bom yes) (on_board yes)
-    (property "Reference" "#PWR0176" (id 0) (at 147.955 45.085 0)
+    (property "Reference" "#PWR078" (id 0) (at 147.955 45.085 0)
       (effects (font (size 1.27 1.27)) hide)
     )
@@
   (symbol (lib_id "power:GND") (at 142.24 51.435 0) (unit 1)
     (in_bom yes) (on_board yes)
-    (property "Reference" "#PWR0175" (id 0) (at 142.24 57.785 0)
+    (property "Reference" "#PWR077" (id 0) (at 142.24 57.785 0)
       (effects (font (size 1.27 1.27)) hide)
     )
@@
   (symbol (lib_id "Device:R") (at 118.745 80.01 0) (unit 1)
     (in_bom yes) (on_board yes)
-    (property "Reference" "R37" (id 0) (at 116.205 81.28 90)
-      (effects (font (size 1.27 1.27)) (justify left))
-    )
-    (property "Value" "10k" (id 1) (at 118.745 81.915 90)
+    (property "Reference" "R36" (id 0) (at 113.03 78.74 0)
+      (effects (font (size 1.27 1.27)) (justify left))
+    )
+    (property "Value" "10k" (id 1) (at 113.03 81.28 0)
       (effects (font (size 1.27 1.27)) (justify left))
     )
@@
   (symbol (lib_id "power:GND") (at 196.215 88.265 0) (unit 1)
     (in_bom yes) (on_board yes)
-    (property "Reference" "#PWR0177" (id 0) (at 196.215 94.615 0)
+    (property "Reference" "#PWR081" (id 0) (at 196.215 94.615 0)
       (effects (font (size 1.27 1.27)) hide)
     )
@@
   (symbol (lib_id "Connector:DB9_Female") (at 159.385 132.08 0) (mirror y) (unit 1)
     (in_bom yes) (on_board yes)
-    (property "Reference" "J22" (id 0) (at 159.385 149.86 0))
-    (property "Value" "DB9_Female_DCE" (id 1) (at 161.4678 147.3454 0))
+    (property "Reference" "J26" (id 0) (at 159.385 149.86 0))
+    (property "Value" "RS_232" (id 1) (at 161.4678 147.3454 0))
     (property "Footprint" "Connector_Dsub:DSUB-9_Female_Horizontal_P2.77x2.84mm_EdgePinOffset7.70mm_Housed_MountingHolesOffset9.12mm" (id 2) (at 159.385 132.08 0)
       (effects (font (size 1.27 1.27)) hide)
@@
   (symbol (lib_id "power:GND") (at 202.565 80.645 0) (unit 1)
     (in_bom yes) (on_board yes)
-    (property "Reference" "#PWR0178" (id 0) (at 202.565 86.995 0)
+    (property "Reference" "#PWR082" (id 0) (at 202.565 86.995 0)
       (effects (font (size 1.27 1.27)) hide)
     )
@@
   (symbol (lib_id "power:GND") (at 147.955 113.03 0) (unit 1)
     (in_bom yes) (on_board yes)
-    (property "Reference" "#PWR0180" (id 0) (at 147.955 119.38 0)
-      (effects (font (size 1.27 1.27)) hide)
-    )
+    (property "Reference" "#PWR079" (id 0) (at 147.955 119.38 0)
+      (effects (font (size 1.27 1.27)) hide)
+    )
