File: handcart.kicad_pcb (KiCad board)
At the start: 2 copper layers, 116 parts, among them J1 Conn_01x05, J10 Conn_02x03_Odd_Even, J11 Conn_01x03, J12 Conn_01x04, J13 Conn_01x04, J132 TE_Ampseal_23, J14 Conn_01x03, J15 Conn_01x02, J16 Conn_01x02, J17 Conn_01x02, J18 Conn_01x02, J19 Raspberry_Pi_2_3, J2 Conn_01x02, J20 Conn_01x02, J21 Conn_01x02, J22 DB9_Female_DCE, J23 Conn_02x05, J24 TE_AmpSeal_14_776273-1, J25 Conn_02x06_Top_Bottom, J3 Conn_01x02, J4 Conn_01x02, J5 Conn_01x02, J6 Conn_01x02, J7 Conn_01x02, J8 Conn_01x02, J9 Conn_01x02, K1 EX12U1S, Q1 2N7002NXAK, Q10 SSM3K361TU,LF, Q11 SSM3K361TU,LF, Q12 2N7002NXAKR, Q13 NTR5105PT1G, Q14 SSM3K361TU,LF, Q15 2N7002NXAK, Q2 NTR5105PT1G, Q3 NTR5105PT1G, Q4 SSM3K361TU,LF, Q5 SSM3K361TU,LF, Q6 2N7002NXAK, Q7 SSM3K361TU,LF, Q8 SSM3K361TU,LF, Q9 SSM3K361TU,LF, SW1 SW_SPDT, U1 Tex_DCDC_v2, U2 DCDC2510, U3 PCA9634PW,118, U4 MCP2515-xSO, U5 MCP2562-E-SN, U6 MAX3232CDR, Y1 16MHz

Commit message: modified schematic and started design pcb
Parts:
- removed D7: SMAJ40CA, Diode_SMD:D_SMA
- removed J132: TE_Ampseal_23, Eagle_Connectors:TE_1-776228-4
- removed the Q6 at (271.8, 111.8)
- removed the Q6 at (257.8, 75.2)
- removed R120: R, Resistor_SMD:R_0805_2012Metric
- added BZ1: Buzzer, Buzzer_Beeper:Buzzer_TDK_PS1240P02BT_D12.2mm_H6.5mm, F.Cu at (182.9, 213.4)
- added C11: 100nF, Resistor_SMD:R_0805_2012Metric, F.Cu at (231.1, 115.3)
- added C12: 100nF, Resistor_SMD:R_0805_2012Metric, F.Cu at (185.4, 149.9)
- added C13: 100nF, Resistor_SMD:R_0805_2012Metric, F.Cu at (181.6, 153.7)
- added C14: 100nF, Resistor_SMD:R_0805_2012Metric, F.Cu at (241.3, 116.0)
- added C15: 2pF, Resistor_SMD:R_0603_1608Metric, F.Cu at (207.8, 185.0)
- added C16: 2pF, Resistor_SMD:R_0603_1608Metric, F.Cu at (209.4, 185.0)
- added C17: 2pF, Resistor_SMD:R_0603_1608Metric, F.Cu at (210.9, 185.0)
- added C18: C, Resistor_SMD:R_0805_2012Metric, F.Cu at (212.4, 208.5)
- added C19: 2pF, Resistor_SMD:R_0603_1608Metric, F.Cu at (212.4, 185.0)
- added C20: 2pF, Resistor_SMD:R_0603_1608Metric, F.Cu at (212.5, 197.9)
- added C21: 2pF, Resistor_SMD:R_0603_1608Metric, F.Cu at (205.8, 189.8)
- added C22: C, Resistor_SMD:R_0805_2012Metric, F.Cu at (216.4, 199.9)
- added C23: 2pF, Resistor_SMD:R_0603_1608Metric, F.Cu at (207.3, 189.8)
- added C24: 2pF, Resistor_SMD:R_0603_1608Metric, F.Cu at (208.8, 189.8)
- added C25: 2pF, Resistor_SMD:R_0603_1608Metric, F.Cu at (212.5, 201.2)
- added C26: C, Resistor_SMD:R_0805_2012Metric, F.Cu at (220.5, 199.9)
- added C27: 2pF, Resistor_SMD:R_0603_1608Metric, F.Cu at (210.4, 189.8)
- added C28: 10uF, Resistor_SMD:R_0603_1608Metric, F.Cu at (226.9, 195.6)
- added C29: C, Resistor_SMD:R_0805_2012Metric, F.Cu at (224.5, 199.9)
- added C30: 10uF, Resistor_SMD:R_0603_1608Metric, F.Cu at (225.9, 188.3)
- added C31: 10uF, Resistor_SMD:R_0603_1608Metric, F.Cu at (225.9, 191.4)
- added C32: 2pF, Resistor_SMD:R_0603_1608Metric, F.Cu at (212.5, 204.7)
- added C33: 0.1uF, Resistor_SMD:R_0603_1608Metric, F.Cu at (227.8, 188.1)
- added C34: 0.1uF, Resistor_SMD:R_0603_1608Metric, F.Cu at (227.8, 191.4)
- added C35: C, Resistor_SMD:R_0805_2012Metric, F.Cu at (230.6, 199.9)
- added D10: 3V3, Resistor_SMD:R_0805_2012Metric, F.Cu at (208.9, 214.0)
- added D11: BAT54S, Package_TO_SOT_SMD:SOT-23, F.Cu at (147.4, 228.2)
- added D12: BAT54S, Package_TO_SOT_SMD:SOT-23, F.Cu at (303.0, 199.1)
- added D13: BAT54S, Package_TO_SOT_SMD:SOT-23, F.Cu at (253.0, 206.8)
- added D14: BAT54S, Package_TO_SOT_SMD:SOT-23, F.Cu at (293.1, 202.9)
- added D15: BAT54S, Package_TO_SOT_SMD:SOT-23, F.Cu at (312.4, 206.4)
- added D16: DDZ13ASF 13V, Diode_SMD:D_SOD-323F, F.Cu at (302.3, 205.7)
- added D17: 1N4148W, Diode_SMD:D_SOD-323_HandSoldering, F.Cu at (185.4, 203.2)
- added D18: BAT54S, Package_TO_SOT_SMD:SOT-23, F.Cu at (384.5, 125.3)
- added D19: SMAJ40CA, Diode_SMD:D_SMA, F.Cu at (358.7, 144.7)
- added D8: VSD, Resistor_SMD:R_0805_2012Metric, F.Cu at (202.6, 214.0)
- added D9: 5V, Resistor_SMD:R_0805_2012Metric, F.Cu at (205.7, 214.0)
- added F1: 10A, Eagle_Main:Keystone-Fuseholder 3557-2, F.Cu at (147.4, 214.2)
- added F2: 5A, Eagle_Main:Keystone-Fuseholder 3557-2, F.Cu at (157.6, 214.2)
- added F3: 2A, Eagle_Main:Keystone-Fuseholder 3557-2, F.Cu at (167.7, 214.2)
- added IC1: MAX11337ATJ+, 00_proj-lib:QFN50P500X500X80-33N, F.Cu at (220.8, 190.2)
- added J26: RS_232, Connector_Dsub:DSUB-9_Female_Horizontal_P2.77x2.84mm_EdgePinOffset7.70mm_Housed_MountingHolesOffset9.12mm, F.Cu at (184.3, 227.3)
- added J27: DISCHARGE_RELAY, Connector_Molex:Molex_Micro-Fit_3.0_43650-0200_1x02_P3.00mm_Horizontal, F.Cu at (332.6, 185.4)
- added J28: ADD_RGB_STRIP, Connector_Molex:Molex_Micro-Fit_3.0_43650-0315_1x03_P3.00mm_Vertical, F.Cu at (226.5, 121.5)
- added J29: SPARE_ADC, Connector_Molex:Molex_Micro-Fit_3.0_43045-0612_2x03_P3.00mm_Vertical, F.Cu at (217.8, 223.1)
- added J30: SD_END_TEST_POINT, Connector_Molex:Molex_Micro-Fit_3.0_43650-0215_1x02_P3.00mm_Vertical, F.Cu at (302.1, 129.8)
- added JP2: 3V3_RASPI, Jumper:SolderJumper-2_P1.3mm_Open_RoundedPad1.0x1.5mm, F.Cu at (181.6, 149.9)
- added JP3: 5V_ADD_STRIP, Jumper:SolderJumper-2_P1.3mm_Open_RoundedPad1.0x1.5mm, F.Cu at (231.8, 125.7)
- added JP4: 3V3_ADD_STRIP, Jumper:SolderJumper-2_P1.3mm_Open_RoundedPad1.0x1.5mm, F.Cu at (231.8, 123.2)
- added Q16: 2N7002NXAK, Package_TO_SOT_SMD:SOT-23, F.Cu at (193.0, 208.3)
- added Q6: SSM3K361TU,LF, 00_proj-lib:SOTFL65P210X75-3N, F.Cu at (244.3, 105.4)
- added R45: 330k, Resistor_SMD:R_0603_1608Metric, F.Cu at (372.8, 139.4)
- added R46: 2k2, Resistor_SMD:R_0603_1608Metric, F.Cu at (194.9, 217.8)
- added R47: 1k, Resistor_SMD:R_0603_1608Metric, F.Cu at (198.8, 217.6)
- added R48: 1k, Resistor_SMD:R_0603_1608Metric, F.Cu at (202.6, 217.6)
- added R49: 270R, Resistor_SMD:R_0603_1608Metric, F.Cu at (205.7, 217.6)
- added R50: 330R, Resistor_SMD:R_0603_1608Metric, F.Cu at (208.9, 217.6)
- added R51: 22R, Resistor_SMD:R_0603_1608Metric, F.Cu at (195.6, 203.2)
- added R52: 330k, Resistor_SMD:R_0603_1608Metric, F.Cu at (193.0, 203.2)
- added R53: R, Resistor_SMD:R_0805_2012Metric, F.Cu at (208.9, 206.5)
- added R54: R, Resistor_SMD:R_0805_2012Metric, F.Cu at (212.4, 206.5)
- added R55: 47k, Resistor_SMD:R_0603_1608Metric, F.Cu at (209.2, 196.1)
- added R56: 47k, Resistor_SMD:R_0603_1608Metric, F.Cu at (212.5, 196.2)
- added R57: R, Resistor_SMD:R_0805_2012Metric, F.Cu at (218.4, 203.5)
- added R58: R, Resistor_SMD:R_0805_2012Metric, F.Cu at (218.4, 199.9)
- added R59: 47k, Resistor_SMD:R_0603_1608Metric, F.Cu at (209.3, 199.4)
- added R60: 47k, Resistor_SMD:R_0603_1608Metric, F.Cu at (212.6, 199.4)
- added R61: R, Resistor_SMD:R_0805_2012Metric, F.Cu at (222.5, 203.5)
- added R62: R, Resistor_SMD:R_0805_2012Metric, F.Cu at (222.5, 199.9)
- added R63: 47k, Resistor_SMD:R_0603_1608Metric, F.Cu at (226.9, 193.9)
- added R64: R, Resistor_SMD:R_0805_2012Metric, F.Cu at (226.6, 203.5)
- added R65: R, Resistor_SMD:R_0805_2012Metric, F.Cu at (226.6, 199.9)
- added R66: 47k, Resistor_SMD:R_0603_1608Metric, F.Cu at (209.5, 202.7)
- added R67: 47k, Resistor_SMD:R_0603_1608Metric, F.Cu at (212.5, 202.7)
- added R68: R, Resistor_SMD:R_0805_2012Metric, F.Cu at (230.6, 203.5)
- added R69: R, Resistor_SMD:R_0805_2012Metric, F.Cu at (228.6, 199.9)
- added R70: R, Resistor_SMD:R_0805_2012Metric, F.Cu at (368.6, 139.6)
- added RN3: 47k, Resistor_SMD:R_Array_Convex_4x0603, F.Cu at (215.1, 185.6)
- added RN4: 47k, Resistor_SMD:R_Array_Convex_4x0603, F.Cu at (213.2, 189.3)
- added RN5: 470k, Resistor_SMD:R_Array_Convex_4x0603, F.Cu at (215.1, 180.5)
- added RN6: 470k, Resistor_SMD:R_Array_Convex_4x0603, F.Cu at (213.2, 193.7)
- added TP1: TP_3V3, TestPoint:TestPoint_Pad_D2.0mm, F.Cu at (174.6, 151.1)
- added TP2: TP_5V, TestPoint:TestPoint_Pad_D2.0mm, F.Cu at (176.5, 201.9)
- added TP3: TP_24V, TestPoint:TestPoint_Pad_D2.0mm, F.Cu at (145.4, 201.9)
- added TP4: TP_12V, TestPoint:TestPoint_Pad_D2.0mm, F.Cu at (154.9, 226.7)
- added TP5: TP_VSD, TestPoint:TestPoint_Pad_D2.0mm, F.Cu at (160.7, 226.7)
- added TP6: TP_RASP_SD_CONTROL, TestPoint:TestPoint_Pad_D2.0mm, F.Cu at (389.9, 121.7)
- added TP7: TP_PON_CHARGER, TestPoint:TestPoint_Pad_D2.0mm, F.Cu at (361.6, 149.0)
- D4: value DDZ13ASF 13V -> 24V; footprint Diode_SMD:D_SOD-323F -> Resistor_SMD:R_0805_2012Metric
- D6: value RGL34B -> 12V; footprint Diode_SMD:D_MiniMELF -> Resistor_SMD:R_0805_2012Metric
- J1: value Conn_01x05 -> ROTARY ENCODER
- J10: value Conn_02x03_Odd_Even -> SPARE_SUPPLY
- J11: value Conn_01x03 -> CAN
- J12: value Conn_01x04 -> SPARE_CHARGER; footprint Connector_Molex:Molex_Micro-Fit_3.0_43650-0400_1x04_P3.00mm_Horizontal -> Connector_Molex:Molex_Micro-Fit_3.0_43045-0612_2x03_P3.00mm_Vertical
- J13: value Conn_01x04 -> SPARE_BMS; footprint Connector_Molex:Molex_Micro-Fit_3.0_43650-0400_1x04_P3.00mm_Horizontal -> Connector_Molex:Molex_Micro-Fit_3.0_43045-1012_2x05_P3.00mm_Vertical
- J14: value Conn_01x03 -> ADD_FAN; footprint Connector_Molex:Molex_Micro-Fit_3.0_43650-0315_1x03_P3.00mm_Vertical -> Connector_Molex:Molex_Micro-Fit_3.0_43650-0215_1x02_P3.00mm_Vertical
- J15: value Conn_01x02 -> EXT_SCREEN; footprint Connector_Molex:Molex_Micro-Fit_3.0_43650-0215_1x02_P3.00mm_Vertical -> Connector_Molex:Molex_Micro-Fit_3.0_43650-0315_1x03_P3.00mm_Vertical
- J16: value Conn_01x02 -> CHARGER; footprint Connector_Molex:Molex_Micro-Fit_3.0_43650-0215_1x02_P3.00mm_Vertical -> 00_proj-lib:TE_776266-4
- J17: value Conn_01x02 -> BMS; footprint Connector_Molex:Molex_Micro-Fit_3.0_43650-0215_1x02_P3.00mm_Vertical -> Eagle_Connectors:TE_1-776228-4
- J18: value Conn_01x02 -> SPARE_RASPI; footprint Connector_Molex:Molex_Micro-Fit_3.0_43650-0200_1x02_P3.00mm_Horizontal -> Connector_Molex:Molex_Micro-Fit_3.0_43045-0612_2x03_P3.00mm_Vertical
- J2: value Conn_01x02 -> ARROW_KEYS_1
- J20: value Conn_01x02 -> RASPI_FAN
- J21: value Conn_01x02 -> GREEN_TS_OFF; footprint Connector_Molex:Molex_Micro-Fit_3.0_43650-0215_1x02_P3.00mm_Vertical -> Connector_Molex:Molex_Micro-Fit_3.0_43650-0200_1x02_P3.00mm_Horizontal
- J22: value DB9_Female_DCE -> RED_IMD_FAULT; footprint Connector_Dsub:DSUB-9_Female_Horizontal_P2.77x2.84mm_EdgePinOffset7.70mm_Housed_MountingHolesOffset9.12mm -> Connector_Molex:Molex_Micro-Fit_3.0_43650-0200_1x02_P3.00mm_Horizontal
- J23: value Conn_02x05 -> RED_BMS_FAULT; footprint Connector_Molex:Molex_Micro-Fit_3.0_43045-1012_2x05_P3.00mm_Vertical -> Connector_Molex:Molex_Micro-Fit_3.0_43650-0200_1x02_P3.00mm_Horizontal
- J24: value TE_AmpSeal_14_776273-1 -> RGB_STRIP; footprint 00_proj-lib:TE_776266-4 -> Connector_Molex:Molex_Micro-Fit_3.0_43650-0400_1x04_P3.00mm_Horizontal
- J25: value Conn_02x06_Top_Bottom -> TSAL; footprint Connector_Molex:Molex_Micro-Fit_3.0_43045-1012_2x05_P3.00mm_Vertical -> Connector_Molex:Molex_Micro-Fit_3.0_43650-0400_1x04_P3.00mm_Horizontal
- J3: value Conn_01x02 -> ARROW_KEYS_2
- J4: value Conn_01x02 -> ARROW_KEYS_3
- J5: value Conn_01x02 -> ARROW_KEYS_4
- J6: value Conn_01x02 -> RESET_BUTTON
- J7: value Conn_01x02 -> TSMS
- J8: value Conn_01x02 -> MUSHROOM
- J9: value Conn_01x02 -> POWER_IN
- JP1: value SolderJumper_2_Open -> RASPBERRY_bypass
- Q1: value 2N7002NXAK -> SSM3K361TU,LF; footprint Package_TO_SOT_SMD:SOT-23 -> 00_proj-lib:SOTFL65P210X75-3N
- Q13: value NTR5105PT1G -> 2N7002NXAKR
- Q14, Q4, Q5: value SSM3K361TU,LF -> NTR5105PT1G; footprint 00_proj-lib:SOTFL65P210X75-3N -> Package_TO_SOT_SMD:SOT-23
- Q2, Q3: value NTR5105PT1G -> 2N7002NXAK
- R1: value 10k -> 22R; footprint Resistor_SMD:R_0805_2012Metric -> Resistor_SMD:R_0603_1608Metric
- R10, R11, R9: value R -> 22R; footprint Resistor_SMD:R_1206_3216Metric -> Resistor_SMD:R_0603_1608Metric
- R12, R7: value R -> 330k; footprint Resistor_SMD:R_1206_3216Metric -> Resistor_SMD:R_0603_1608Metric
- R13: value 33 -> 330k
- R14: value 10k -> 330k
- R15, R16, R17: value 22 -> 120R
- R18, R19, R24, R30, R42, R44: value 330k -> 22R
- R2: value 10k -> 330k; footprint Resistor_SMD:R_0805_2012Metric -> Resistor_SMD:R_0603_1608Metric
- R21, R27, R33, R41, R43: value 22 -> 330k
- R22, R28, R34: value 330k -> R; footprint Resistor_SMD:R_0603_1608Metric -> Resistor_SMD:R_0805_2012Metric
- R23, R29, R35: value 22 -> R; footprint Resistor_SMD:R_0603_1608Metric -> Resistor_SMD:R_0805_2012Metric
- R25, R31, R39: value 22 -> 22R
- R3: value 10k -> 4k7; footprint Resistor_SMD:R_0805_2012Metric -> Resistor_SMD:R_0603_1608Metric
- R36: value 330k -> 10k
- R38: value 10k -> 22R
- R4, R5: value 120R -> 4k7; footprint Resistor_SMD:R_2512_6332Metric -> Resistor_SMD:R_0603_1608Metric
- R6: value 120R -> 22R; footprint Resistor_SMD:R_2512_6332Metric -> Resistor_SMD:R_0603_1608Metric
- R8: value R -> 120R; footprint Resistor_SMD:R_1206_3216Metric -> Resistor_SMD:R_0603_1608Metric
- RN1, RN2: footprint Resistor_SMD:R_Array_Convex_4x0612 -> Resistor_SMD:R_Array_Convex_4x0603
- moved J14 186.6 mm to (396.8, 168.7), turned to 0 degrees
- moved RN2 165.7 mm to (372.0, 183.9)
- moved R1 164.0 mm to (395.1, 155.6)
- moved J5 154.0 mm to (386.0, 177.0), turned to 0 degrees
- moved C10 147.7 mm to (195.7, 222.0), turned to 90 degrees
- moved C7 145.7 mm to (205.5, 223.3), turned to -90 degrees
- moved SW1 145.1 mm to (202.9, 237.0), turned to 0 degrees
- moved R37 142.7 mm to (205.5, 228.4), turned to -90 degrees
- moved U6 140.5 mm to (200.4, 227.1)
- moved C6 136.9 mm to (193.3, 223.0), turned to -90 degrees
- moved D1 135.6 mm to (380.1, 193.3)
- moved D6 133.4 mm to (198.8, 214.0), turned to -90 degrees
- moved C9 133.1 mm to (195.7, 228.5), turned to 90 degrees
- moved C8 128.2 mm to (195.6, 225.6), turned to -90 degrees
- moved R36 127.0 mm to (207.3, 229.1), turned to -90 degrees
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Connections:
- net /RS_232/RASP_RX renamed /RS_232+FEEDBACK/RASP_RX
- net /RS_232/RASP_TX_RS232 renamed /RS_232+FEEDBACK/RASP_TX_RS232
- D1 pad 1: +5V -> +24V
- D2 pad 1: +24V -> +5V
- D3 pad 2: Net-(D3-Pad2) -> /Shutdown+Discharge/RELE_SHUTDOWN_FB
- D4 pad 1: /SD_END -> GND
- D4 pad 2: GND -> Net-(D4-Pad2)
- D5 pad 1: /SD_END_HV -> Net-(D18-Pad3)
- D6 pad 1: /DISCHARGE_P -> GND
- D6 pad 2: /SD_BMS_OUT -> Net-(D6-Pad2)
- J10 pad 1: /NC_CRG_1 -> +24V
- J10 pad 2: /NC_CRG_2 -> +5V
- J10 pad 3: /NC_CRG_3 -> +12V
- J10 pad 4: unconnected-(J10-Pad4) -> +3V3
- J10 pad 5: unconnected-(J10-Pad5) -> GND
- J10 pad 6: unconnected-(J10-Pad6) -> GND
- J11 pad 1: /CAN_P -> Net-(J11-Pad1)
- J11 pad 2: /CAN_N -> Net-(J11-Pad2)
- J12 pad 1: +12V -> /NC_CRG_1
- J12 pad 2: /TSAL_R -> /NC_CRG_2
- J12 pad 3: /TSAL_G -> /NC_CRG_3
- J12 pad 4: /TSAL_B -> /NC_CRG_4
- J13 pad 1: +12V -> /NC_BMS_1
- J13 pad 2: /STRIP1_R -> /NC_BMS_2
- J13 pad 3: /STRIP1_G -> /NC_BMS_3
- J13 pad 4: /STRIP1_B -> /NC_BMS_4
- J14 pad 1: +5V -> +24V
- J14 pad 2: +3V3 -> Net-(D1-Pad2)
- J15 pad 2: /GREEN_TS_OFF -> +3V3
- J16 pad 1: /RED_BMS_FAULT -> /CAN_P
- J16 pad 2: GND -> /CAN_N
- J17 pad 1: /RED_IMD_FAULT -> +24V
- J17 pad 2: GND -> +24V
- J18 pad 1: /DISCHARGE_P -> /Raspberry/NC_RASP_1
- J18 pad 2: /DISCHARGE_N -> /Raspberry/NC_RASP_2
- J19 pad 1: +3V3 -> Net-(J19-Pad1)
- J19 pad 12: /Raspberry/NC_RASP_8 -> /Raspberry/ADD_RGB_STRIP
- J19 pad 17: +3V3 -> Net-(J19-Pad1)
- J19 pad 24: /Raspberry/RASP_~{CS} -> /Raspberry/RASP_MOSI
- J19 pad 28: /Raspberry/NC_RASP_7 -> /Raspberry/BUZZER
- J19 pad 35: /RASP_PON_CHARGER -> /RASP_PON_DISCHARGER
- J19 pad 8: /RS_232/RASP_TX -> /RS_232+FEEDBACK/RASP_TX
- J20 pad 2: Net-(D1-Pad2) -> Net-(D2-Pad2)
- J21 pad 1: +24V -> +5V
- J21 pad 2: Net-(D2-Pad2) -> Net-(J21-Pad2)
- J22 pad 1: unconnected-(J22-Pad1) -> Net-(J22-Pad1)
- J22 pad 2: /BRUSA_TX -> GND
- J23 pad 1: /NC_BMS_1 -> Net-(R17-Pad2)
- J23 pad 2: /NC_BMS_2 -> GND
- J24 pad 1: /CAN_P -> +12V
- J24 pad 2: /CAN_N -> /Output/STRIP1_R
- J24 pad 3: /BRUSA_TX -> /Output/STRIP1_G
- J24 pad 4: /BRUSA_RX -> /Output/STRIP1_B
- J25 pad 1: /Raspberry/NC_RASP_1 -> +24V
- J25 pad 2: /Raspberry/NC_RASP_2 -> /Output/TSAL_R
- J25 pad 3: /Raspberry/NC_RASP_3 -> /Output/TSAL_G
- J25 pad 4: /Raspberry/NC_RASP_4 -> /Output/TSAL_B
- J8 pad 1: +24V -> /SD_TO_MUSHROOM
- J8 pad 2: /SD_FROM_MUSHROOM -> /SD_TO_CHARGER
- J9 pad 1: +24V -> Net-(D11-Pad3)
- K1 pad 1: /SD_FROM_MUSHROOM -> VCC
- K1 pad 2: Net-(D3-Pad2) -> /Shutdown+Discharge/RELE_SHUTDOWN_FB
- K1 pad 4: /SD_TO_CHARGER -> /SD_TO_MUSHROOM
- Q1 pad 3: Net-(Q1-Pad3) -> Net-(D1-Pad2)
- Q10 pad 1: Net-(R29-Pad1) -> Net-(Q10-Pad1)
- Q10 pad 3: Net-(R11-Pad1) -> Net-(Q10-Pad3)
- Q11 pad 1: Net-(R31-Pad1) -> Net-(Q11-Pad1)
- Q13 pad 2: /SD_END -> GND
- Q13 pad 3: /PON -> /Shutdown+Discharge/RELE_SHUTDOWN_FB
- Q14 pad 1: Net-(R43-Pad1) -> Net-(Q14-Pad1)
- Q14 pad 2: GND -> /SD_END
- Q14 pad 3: Net-(D3-Pad2) -> /PON
- Q15 pad 3: /DISCHARGE_N -> /Shutdown+Discharge/COIL_DISCHARGE_FB
- Q2 pad 2: +5V -> GND
- Q2 pad 3: Net-(Q2-Pad3) -> Net-(D2-Pad2)
- Q3 pad 2: +5V -> GND
- Q4 pad 1: Net-(R21-Pad1) -> Net-(Q4-Pad1)
- Q4 pad 2: GND -> +5V
- Q4 pad 3: Net-(R7-Pad1) -> Net-(Q4-Pad3)
- Q5 pad 1: Net-(R23-Pad1) -> Net-(Q5-Pad1)
- Q5 pad 2: GND -> +5V
- Q5 pad 3: Net-(R8-Pad1) -> Net-(Q5-Pad3)
- Q7 pad 1: Net-(R25-Pad1) -> Net-(Q7-Pad1)
- Q8 pad 1: Net-(R27-Pad1) -> Net-(Q8-Pad1)
- Q8 pad 3: Net-(R10-Pad1) -> Net-(Q8-Pad3)
- Q9 pad 1: Net-(R35-Pad1) -> Net-(Q9-Pad1)
- Q9 pad 3: Net-(D2-Pad2) -> Net-(Q9-Pad3)
- R1 pad 1: +3V3 -> Net-(Q1-Pad1)
- R1 pad 2: /Raspberry/SDA -> /ADD_FAN_PWM
- R10 pad 1: Net-(R10-Pad1) -> /IMD_LED
- R10 pad 2: /STRIP1_R -> Net-(Q4-Pad1)
- R11 pad 1: Net-(R11-Pad1) -> /BMS_LED
- R11 pad 2: /STRIP1_G -> Net-(Q5-Pad1)
- R12 pad 1: Net-(Q11-Pad3) -> Net-(Q3-Pad1)
- R12 pad 2: /STRIP1_B -> GND
- R13 pad 1: Net-(Q15-Pad1) -> Net-(Q4-Pad1)
- R13 pad 2: /RASP_PON_CHARGER -> GND
- R14 pad 1: Net-(Q15-Pad1) -> Net-(Q5-Pad1)
- R15 pad 1: /TSAL -> Net-(Q3-Pad3)
- R15 pad 2: Net-(Q1-Pad1) -> Net-(J21-Pad2)
- R16 pad 1: /IMD_LED -> Net-(Q4-Pad3)
- R16 pad 2: Net-(Q2-Pad1) -> Net-(J22-Pad1)
- R17 pad 1: /BMS_LED -> Net-(Q5-Pad3)
- R17 pad 2: Net-(Q3-Pad1) -> Net-(R17-Pad2)
- R18 pad 1: Net-(Q1-Pad1) -> Net-(Q6-Pad1)
- R18 pad 2: GND -> /Output/RASPY_TSAL_R
- R19 pad 1: Net-(Q2-Pad1) -> Net-(Q7-Pad1)
- R19 pad 2: GND -> /Output/RASPY_STRIP1_R
- R2 pad 1: +3V3 -> Net-(Q1-Pad1)
- R2 pad 2: /Raspberry/SCL -> GND
- R20 pad 1: Net-(Q3-Pad1) -> Net-(Q6-Pad1)
- R21 pad 1: Net-(R21-Pad1) -> Net-(Q7-Pad1)
- R21 pad 2: /Output/RASPY_TSAL_R -> GND
- R22 pad 1: Net-(R21-Pad1) -> Net-(Q6-Pad3)
- R22 pad 2: GND -> /Output/TSAL_R
- R23 pad 1: Net-(R23-Pad1) -> Net-(Q7-Pad3)
- R23 pad 2: /Output/RASPY_TSAL_G -> /Output/STRIP1_R
- R24 pad 1: Net-(R23-Pad1) -> Net-(Q9-Pad1)
- R24 pad 2: GND -> /Output/RASPY_TSAL_G
- R25 pad 1: Net-(R25-Pad1) -> Net-(Q8-Pad1)
- R25 pad 2: /Output/RASPY_TSAL_B -> /Output/RASPY_STRIP1_G
- R26 pad 1: Net-(R25-Pad1) -> Net-(Q9-Pad1)
- R27 pad 1: Net-(R27-Pad1) -> Net-(Q8-Pad1)
- R27 pad 2: /Output/RASPY_STRIP1_R -> GND
- R28 pad 1: Net-(R27-Pad1) -> Net-(Q8-Pad3)
- R28 pad 2: GND -> /Output/STRIP1_G
- R29 pad 1: Net-(R29-Pad1) -> Net-(Q9-Pad3)
- R29 pad 2: /Output/RASPY_STRIP1_G -> /Output/TSAL_G
- R3 pad 2: /Raspberry/~{OE} -> /Raspberry/SDA
- R30 pad 1: Net-(R29-Pad1) -> Net-(Q10-Pad1)
- R30 pad 2: GND -> /Output/RASPY_TSAL_B
- R31 pad 1: Net-(R31-Pad1) -> Net-(Q11-Pad1)
- R32 pad 1: Net-(R31-Pad1) -> Net-(Q10-Pad1)
- R33 pad 1: Net-(R33-Pad1) -> Net-(Q11-Pad1)
- R33 pad 2: /Output/RASPY_FAN_PWM -> GND
- R34 pad 1: Net-(R33-Pad1) -> Net-(Q10-Pad3)
- R34 pad 2: GND -> /Output/TSAL_B
- R35 pad 1: Net-(R35-Pad1) -> Net-(Q11-Pad3)
- R35 pad 2: /Output/ADD_FAN_PWM -> /Output/STRIP1_B
- R36 pad 1: Net-(R35-Pad1) -> +3.3V
- R36 pad 2: GND -> /RS_232+FEEDBACK/RASP_TX
- R37 pad 2: /RS_232/RASP_TX -> Net-(R37-Pad2)
- R38 pad 1: +3.3V -> Net-(Q12-Pad1)
- R38 pad 2: Net-(R38-Pad2) -> /RASP_SD_CONTROL
- R39 pad 1: Net-(Q12-Pad1) -> Net-(Q13-Pad1)
- R39 pad 2: /RASP_SD_CONTROL -> /RASP_PON_CONTROL
- R4 pad 1: Net-(Q1-Pad3) -> +3V3
- R4 pad 2: /GREEN_TS_OFF -> /Raspberry/SCL
- R41 pad 2: Net-(Q12-Pad3) -> GND
- R42 pad 1: /SD_END -> Net-(Q14-Pad1)
- R42 pad 2: Net-(Q13-Pad1) -> Net-(Q12-Pad3)
- R43 pad 1: Net-(R43-Pad1) -> /SD_END
- R43 pad 2: /RASP_PON_CONTROL -> Net-(Q14-Pad1)
- R44 pad 1: Net-(R43-Pad1) -> /RASP_PON_DISCHARGER
- R44 pad 2: GND -> Net-(Q15-Pad1)
- R5 pad 1: /RED_BMS_FAULT -> +3V3
- R5 pad 2: Net-(Q2-Pad3) -> /Raspberry/~{OE}
- R6 pad 1: /RED_IMD_FAULT -> Net-(Q2-Pad1)
- R6 pad 2: Net-(Q3-Pad3) -> /Raspberry/RASPY_FAN_PWM
- R7 pad 1: Net-(R7-Pad1) -> Net-(Q2-Pad1)
- R7 pad 2: /TSAL_R -> GND
- R8 pad 1: Net-(R8-Pad1) -> Net-(J11-Pad1)
- R8 pad 2: /TSAL_G -> Net-(J11-Pad2)
- R9 pad 1: Net-(Q7-Pad3) -> /TSAL
- R9 pad 2: /TSAL_B -> Net-(Q3-Pad1)
- SW1 pad 3: /RS_232/PC_TX -> /RS_232+FEEDBACK/PC_TX
- U2 pad 11: +12V -> Net-(F2-Pad1)
- U2 pad 12: +12V -> Net-(F2-Pad1)
- U2 pad 13: +12V -> Net-(F2-Pad1)
- U2 pad 14: +12V -> Net-(F2-Pad1)
- U3 pad 11: /Output/ADD_FAN_PWM -> /Raspberry/ADD_FAN_PWM
- U3 pad 12: /Output/RASPY_FAN_PWM -> /Raspberry/RASPY_FAN_PWM
- U4 pad 16: /Raspberry/RASP_~{CS} -> /Raspberry/RASP_MOSI
- U5 pad 6: /CAN_N -> Net-(J11-Pad2)
- U5 pad 7: /CAN_P -> Net-(J11-Pad1)
- U6 pad 10: /RS_232/RASP_TX -> /RS_232+FEEDBACK/RASP_TX
- U6 pad 11: Net-(R38-Pad2) -> Net-(R37-Pad2)
Routing:
- net GND: track 0.00 -> 765.5 mm, vias 0 -> 12
- net +5V: track 0.00 -> 273.3 mm
- net +24V: track 0.00 -> 259.2 mm, vias 0 -> 1
- net +3V3: track 0.00 -> 250.4 mm, vias 0 -> 4
- net +12V: track 0.00 -> 226.2 mm, vias 0 -> 2
- net /BRUSA_TX: track 0.00 -> 102.5 mm
- net /Raspberry/SCL: track 0.00 -> 79.9 mm, vias 0 -> 2
- net /Raspberry/~{OE}: track 0.00 -> 79.8 mm, vias 0 -> 2
- net /Raspberry/SDA: track 0.00 -> 77.5 mm, vias 0 -> 2
- net /BRUSA_RX: track 0.00 -> 76.8 mm
- net Net-(F2-Pad1): track 0.00 -> 61.8 mm
- net /PON: track 0.00 -> 59.9 mm, vias 0 -> 2
- net /Raspberry/RASPY_FAN_PWM: track 0.00 -> 59.9 mm, vias 0 -> 2
- net /Raspberry/RASP_CLK: track 0.00 -> 59.2 mm
- net VCC: track 0.00 -> 43.8 mm
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Other:
- board outline added: 213.4 x 156.2 mm

Commit message: First version of the pcb layout
Parts:
- removed C15, C16, C17, C19, C21, C23, C24, C27: 2pF, Resistor_SMD:R_0603_1608Metric
- removed D18: BAT54S, Package_TO_SOT_SMD:SOT-23
- removed D19: SMAJ40CA, Diode_SMD:D_SMA
- added CN1: 100nF, Resistor_SMD:R_Array_Concave_4x0603, F.Cu at (203.5, 148.5)
- added CN2: 100nF, Resistor_SMD:R_Array_Concave_4x0603, F.Cu at (195.5, 154.6)
- added Q17: FQP17P06, Package_TO_SOT_THT:TO-220-3_Vertical, F.Cu at (118.8, 173.4)
- added R71: 1k, Resistor_SMD:R_0603_1608Metric, F.Cu at (124.7, 170.6)
- C20, C25, C32: value 2pF -> 100nF
- C28: value 10uF -> 100n
- D11: value BAT54S -> DDZ3V3ASF-7; footprint Package_TO_SOT_SMD:SOT-23 -> Diode_SMD:D_SOD-323
- J11: footprint Connector_Molex:Molex_Micro-Fit_3.0_43650-0300_1x03_P3.00mm_Horizontal -> Connector_Molex:Molex_Micro-Fit_3.0_43650-0315_1x03_P3.00mm_Vertical
- J17: footprint Eagle_Connectors:TE_1-776228-4 -> Eagle_Connectors:TE_776087-4
- J21, J22, J23, J27: footprint Connector_Molex:Molex_Micro-Fit_3.0_43650-0200_1x02_P3.00mm_Horizontal -> Connector_Molex:Molex_Micro-Fit_3.0_43650-0215_1x02_P3.00mm_Vertical
- J24, J25: footprint Connector_Molex:Molex_Micro-Fit_3.0_43650-0400_1x04_P3.00mm_Horizontal -> Connector_Molex:Molex_Micro-Fit_3.0_43650-0415_1x04_P3.00mm_Vertical
- R46: value 2k2 -> 22k
- R47, R48: value 1k -> 10k
- R49: value 270R -> 2k7
- R50: value 330R -> 2k7
- R55, R59, R66: value 47k -> 27k
- R56, R60, R67, RN3, RN4: value 47k -> 3k3
- RN5, RN6: value 470k -> 27k
- moved J6 284.6 mm to (119.6, 96.7), turned to 180 degrees
- moved J8 245.9 mm to (131.5, 96.7), turned to 180 degrees
- moved J14 235.9 mm to (161.8, 149.8)
- moved R1 225.1 mm to (170.1, 151.1), turned to 180 degrees
- moved D1 216.1 mm to (169.4, 145.2), turned to -90 degrees
- moved R44 196.5 mm to (182.4, 136.7), turned to -90 degrees
- moved Q15 195.9 mm to (177.8, 136.7), turned to 180 degrees
- moved R45 192.2 mm to (180.6, 136.7), turned to 90 degrees
- moved D5 191.4 mm to (178.3, 139.7)
- moved D3 172.4 mm to (212.8, 130.1)
- moved TP6 165.8 mm to (224.5, 134.6)
- moved J27 165.7 mm to (173.3, 139.7), turned to 90 degrees
- moved J30 162.0 mm to (143.5, 96.7), turned to 180 degrees
- moved R41 158.3 mm to (224.4, 129.6), turned to 180 degrees
- moved J7 153.4 mm to (155.4, 96.7), turned to 180 degrees
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Connections:
- C7 pad 1: +3.3V -> +3V3
- D11 pad 1: GND -> Net-(D11-Pad1)
- D11 pad 2: unconnected-(D11-Pad2) -> Net-(D11-Pad2)
- D13 pad 2: +5V -> +12V
- D3 pad 1: +12V -> VCC
- D3 pad 2: /Shutdown+Discharge/RELE_SHUTDOWN_FB -> /RS_232+FEEDBACK/RELE_SUTHDOWN_FB
- F1 pad 1: Net-(D11-Pad3) -> Net-(D11-Pad1)
- IC1 pad 23: /Raspberry/RASP_MOSI -> /RS_232+FEEDBACK/~{CS}
- J18 pad 6: /Raspberry/NC_RASP_6 -> unconnected-(J18-Pad6)
- J19 pad 12: /Raspberry/ADD_RGB_STRIP -> /Output/ADD_RGB_STRIP
- J19 pad 24: /Raspberry/RASP_MOSI -> /Raspberry/RASP_~{CS}
- J19 pad 27: /Raspberry/NC_RASP_6 -> /RS_232+FEEDBACK/~{CS}
- J24 pad 2: /Output/STRIP1_R -> /Output/STRIP1_B
- J24 pad 4: /Output/STRIP1_B -> /Output/STRIP1_R
- J25 pad 2: /Output/TSAL_R -> /Output/TSAL_B
- J25 pad 4: /Output/TSAL_B -> /Output/TSAL_R
- J27 pad 2: /Shutdown+Discharge/COIL_DISCHARGE_FB -> /RS_232+FEEDBACK/COIL_DISCHARGE_FB
- J9 pad 1: Net-(D11-Pad3) -> Net-(J9-Pad1)
- JP1 pad 1: /SD_FROM_MUSHROOM -> VCC
- K1 pad 2: /Shutdown+Discharge/RELE_SHUTDOWN_FB -> /RS_232+FEEDBACK/RELE_SUTHDOWN_FB
- K1 pad 3: +12V -> VCC
- Q13 pad 3: /Shutdown+Discharge/RELE_SHUTDOWN_FB -> /RS_232+FEEDBACK/RELE_SUTHDOWN_FB
- Q15 pad 3: /Shutdown+Discharge/COIL_DISCHARGE_FB -> /RS_232+FEEDBACK/COIL_DISCHARGE_FB
- R36 pad 1: +3.3V -> +3V3
- R37 pad 1: +3.3V -> +3V3
- R63 pad 1: Net-(C28-Pad1) -> +3V3
- R63 pad 2: +3V3 -> Net-(C28-Pad1)
- R8 pad 1: Net-(J11-Pad1) -> Net-(J11-Pad2)
- R8 pad 2: Net-(J11-Pad2) -> Net-(J11-Pad1)
- RN1 pad 5: /BUT_0 -> /BUT_4
- RN1 pad 6: /BUT_1 -> /BUT_3
- RN1 pad 8: /BUT_3 -> /BUT_1
- RN2 pad 5: /BUT_4 -> /ROT_A
- RN2 pad 6: /ROT_A -> /ROT_B
- RN2 pad 7: /ROT_B -> /BUT_0
- U3 pad 11: /Raspberry/ADD_FAN_PWM -> /ADD_FAN_PWM
- U4 pad 16: /Raspberry/RASP_MOSI -> /Raspberry/RASP_~{CS}
- U5 pad 6: Net-(J11-Pad2) -> Net-(J11-Pad1)
- U5 pad 7: Net-(J11-Pad1) -> Net-(J11-Pad2)
- U6 pad 16: +3.3V -> +3V3
Routing:
- net GND: track 765.5 -> 1199.1 mm, vias 12 -> 21
- net /SD_END: track 3.23 -> 359.8 mm, vias 1 -> 4
- net /SD_BMS_OUT: track 1.23 -> 260.7 mm, vias 1 -> 4
- net /RESET_BUTTON: track 0.00 -> 259.5 mm
- net +3V3: track 250.4 -> 484.4 mm, vias 4 -> 11
- net +5V: track 273.3 -> 507.1 mm, vias 0 -> 9
- net VCC: track 43.8 -> 226.8 mm, vias 0 -> 4
- net +12V: track 226.2 -> 387.0 mm
- net /Raspberry/RASP_MISO: track 0.00 -> 155.5 mm, vias 0 -> 5
- net /Raspberry/RASP_MOSI: track 0.00 -> 153.4 mm, vias 0 -> 5
- net /Raspberry/BUZZER: track 0.00 -> 149.6 mm, vias 0 -> 3
- net /SD_TO_CHARGER: track 8.59 -> 155.1 mm, vias 0 -> 1
- net /IMD_LED: track 0.00 -> 134.6 mm, vias 0 -> 2
- net /TSAL: track 0.00 -> 129.3 mm, vias 0 -> 2
- net /RASP_PON_DISCHARGER: track 0.00 -> 128.7 mm, vias 0 -> 2
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Other:
- board size 213.4 x 156.2 mm -> 213.4 x 100.6 mm

Commit message: Second iteration of the board layout. Need to fix some traces
Parts:
- removed J28: ADD_RGB_STRIP, Connector_Molex:Molex_Micro-Fit_3.0_43650-0315_1x03_P3.00mm_Vertical
- removed SW1: SW_SPDT, Button_Switch_THT:SW_E-Switch_EG1224_SPDT_Angled
- added JP5: Jumper_3_Bridged12, Connector_PinHeader_2.54mm:PinHeader_1x03_P2.54mm_Vertical, F.Cu at (269.5, 151.6)
- added REF**: MountingHole_3.2mm_M3_ISO14580, Eagle_Main:MountingHole_3.2mm_M3_ISO14580, F.Cu at (160.2, 72.5)
- added REF**: MountingHole_3.2mm_M3_ISO14580, Eagle_Main:MountingHole_3.2mm_M3_ISO14580, F.Cu at (218.2, 72.5)
- added REF**: MountingHole_3.2mm_M3_ISO14580, Eagle_Main:MountingHole_3.2mm_M3_ISO14580, F.Cu at (303.3, 98.0)
- added REF**: MountingHole_3.2mm_M3_ISO14580, Eagle_Main:MountingHole_3.2mm_M3_ISO14580, F.Cu at (161.1, 139.1)
- added REF**: MountingHole_3.2mm_M3_ISO14580, Eagle_Main:MountingHole_3.2mm_M3_ISO14580, F.Cu at (218.2, 122.0)
- added REF**: MountingHole_3.2mm_M3_ISO14580, Eagle_Main:MountingHole_3.2mm_M3_ISO14580, F.Cu at (307.9, 146.6)
- added REF**: MountingHole_3.2mm_M3_ISO14580, Eagle_Main:MountingHole_3.2mm_M3_ISO14580, F.Cu at (160.2, 122.0)
- J10: footprint Connector_Molex:Molex_Micro-Fit_3.0_43045-0612_2x03_P3.00mm_Vertical -> Connector_Molex:Molex_Micro-Fit_3.0_43045-1012_2x05_P3.00mm_Vertical
- J19: moved to B.Cu
- J24: value RGB_STRIP -> 1-776279-1; footprint Connector_Molex:Molex_Micro-Fit_3.0_43650-0415_1x04_P3.00mm_Vertical -> Eagle_Connectors:17762791
- J9: value POWER_IN -> 1-776279-1; footprint Connector_Molex:Molex_Micro-Fit_3.0_43650-0200_1x02_P3.00mm_Horizontal -> Eagle_Connectors:17762791
- moved Q17 240.0 mm to (356.7, 141.5), turned to -90 degrees
- moved D11 233.0 mm to (353.8, 145.3), turned to 90 degrees
- moved R71 228.5 mm to (351.8, 145.3), turned to -90 degrees
- moved F1 227.6 mm to (354.8, 126.7)
- moved U2 222.1 mm to (356.2, 107.6)
- moved J9 208.8 mm to (338.6, 153.5), turned to 0 degrees
- moved F2 208.0 mm to (345.2, 126.7)
- moved J10 205.9 mm to (327.4, 152.1), turned to 180 degrees
- moved TP4 195.5 mm to (326.6, 135.9)
- moved TP3 194.7 mm to (329.2, 138.9)
- moved F3 189.3 mm to (336.3, 126.7)
- moved TP5 184.3 mm to (324.1, 138.9)
- moved U1 183.7 mm to (328.4, 100.8), turned to 180 degrees
- moved J13 174.6 mm to (141.1, 136.7), turned to -90 degrees
- moved TP1 169.3 mm to (319.0, 138.9)
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Connections:
- J11 pad 1: Net-(J11-Pad1) -> /CAN_N
- J11 pad 2: Net-(J11-Pad2) -> /CAN_P
- J24 pad 1: +12V -> Net-(J24-Pad1)
- J24 pad 2: /Output/STRIP1_B -> /Output/ADD_RGB_STRIP
- J24 pad 3: /Output/STRIP1_G -> GND
- J24 pad 4: /Output/STRIP1_R -> GND
- J9 pad 2: GND -> Net-(J9-Pad1)
- JP1 pad 2: /SD_TO_CHARGER -> /SD_TO_MUSHROOM
- JP3 pad 1: Net-(J28-Pad1) -> Net-(J24-Pad1)
- JP4 pad 1: Net-(J28-Pad1) -> Net-(J24-Pad1)
- R8 pad 1: Net-(J11-Pad2) -> /CAN_P
- R8 pad 2: Net-(J11-Pad1) -> /CAN_N
- U5 pad 6: Net-(J11-Pad1) -> /CAN_N
- U5 pad 7: Net-(J11-Pad2) -> /CAN_P
Routing:
- net /RESET_BUTTON: track 259.5 -> 36.7 mm
- net /SD_BMS_OUT: track 260.7 -> 67.9 mm, vias 4 -> 0
- net /RASP_PON_CONTROL: track 122.7 -> 305.1 mm, vias 4 -> 1
- net +24V: track 366.6 -> 528.9 mm, vias 3 -> 1
- net +12V: track 387.0 -> 234.7 mm, vias 2 -> 6
- net /Output/ADD_RGB_STRIP: track 74.5 -> 210.2 mm, vias 3 -> 1
- net /RS_232+FEEDBACK/RELE_SUTHDOWN_FB: track 70.6 -> 192.0 mm, vias 1 -> 6
- net /SD_TO_MUSHROOM: track 113.2 -> 228.6 mm, vias 0 -> 1
- net /BUT_3: track 26.6 -> 124.8 mm, vias 0 -> 4
- net /CAN_P: track 71.7 -> 163.1 mm, vias 0 -> 4
- net /CAN_N: track 73.8 -> 164.5 mm, vias 0 -> 4
- net /BMS_LED: track 114.8 -> 27.9 mm, vias 2 -> 0
- net /BUT_2: track 20.5 -> 104.5 mm, vias 0 -> 3
- net GND: track 1199.1 -> 1280.5 mm, vias 21 -> 9
- net /BUT_1: track 34.8 -> 116.0 mm, vias 0 -> 3
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Other:
- board size 213.4 x 100.6 mm -> 225 x 100 mm
