File: Indicators.kicad_sch (KiCad schematic)
At the start: 43 parts, among them J21 GREEN_TS_OFF, J22 RED_IMD_FAULT, J23 RED_BMS_FAULT, J24 1-776279-1, J25 TSAL, Q10 SSM3K361TU,LF, Q11 SSM3K361TU,LF, Q3 2N7002NXAK, Q4 NTR5105PT1G, Q5 NTR5105PT1G, Q6 SSM3K361TU,LF, Q7 SSM3K361TU,LF, Q8 SSM3K361TU,LF, Q9 SSM3K361TU,LF

Commit message: Fixed Schematic, fixed some traces. Still not finished
Parts:
- added C14: 100nF, Capacitor_SMD:C_0603_1608Metric, symbol Device:C
- added U3: PCA9634PW,118, 00_proj-lib:SOP65P640X110-20N, symbol 00_proj-lib:PCA9634PW,118
- J24: footprint Eagle_Connectors:17762791 -> Eagle_Connectors:TE-17762791
- R15, R16, R17: footprint Resistor_SMD:R_0603_1608Metric -> Resistor_SMD:R_0805_2012Metric
Connections:
- net +3V3: now also C14.1, U3.1 (A0), U3.20 (VDD), U3.3 (A2), U3.5 (A4)
- net GND: now also C14.2, U3.10 (VSS), U3.16 (A5), U3.17 (A6), U3.2 (A1), U3.4 (A3)
- net RASPY_STRIP1_B: now also U3.13 (LED6)
- net RASPY_STRIP1_G: now also U3.14 (LED7)
- net RASPY_STRIP1_R: now also U3.9 (LED3)
- net RASPY_TSAL_B: now also U3.8 (LED2)
- net RASPY_TSAL_G: now also U3.7 (LED1)
- net RASPY_TSAL_R: now also U3.6 (LED0)
- new net ADD_FAN_PWM: U3.11 (LED4)
- new net RASPY_FAN_PWM: U3.12 (LED5)
- new net SCL: U3.18 (SCL)
- new net SDA: U3.19 (SDA)
- new net ~{OE}: U3.15 (~{OE})
Other:
- note added: "Address: 0010 101X"
- note added: "LEDs DRIVER"
- moved on the sheet: J21, J22, J23, J24, J25, JP3, JP4, Q10, Q11, Q3, Q4, Q5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
